File: PCB/Macropad.kicad_pcb (KiCad board)
At the start: 2 copper layers, 80 x 94 mm, 34 parts, among them SW1 SW_Push, SW10 RotaryEncoder_Switch, SW2 SW_Push, SW3 SW_Push, SW4 SW_Push, SW5 SW_Push, SW6 SW_Push, SW7 SW_Push, SW8 SW_Push, SW9 SW_Push, U1 MOUDLE-SEEEDUINO-XIAO, U2 ER_OLEDM0.91_1x-I2C

Commit message: Update PCB file
Parts:
- moved U1 7.87 mm to (145.8, 53.8)
Routing:
- net Col 1: track 123.2 -> 141.2 mm
- net SCL: track 27.0 -> 43.7 mm
- net RNB: track 32.5 -> 41.4 mm
- net LED: track 35.0 -> 43.9 mm
- net GND: track 319.8 -> 328.2 mm
- net +5V: track 288.9 -> 297.3 mm
- net Row 2: track 68.3 -> 76.5 mm
- net Col 2: track 124.9 -> 132.8 mm
- net Col 0: track 79.1 -> 86.7 mm
- net Row 1: track 109.0 -> 114.7 mm, vias 5 -> 4
- net RNA: track 48.3 -> 53.9 mm
- net Row 0: track 119.5 -> 122.8 mm
- net SDA: track 27.0 -> 29.7 mm
